Commit message: Interactive UI to visualize visuo-tactile sensors

File: src/robotera_ball_handling/source/robotera_ball_handling/assets/robots/xhand/urdf/robotera_xhand_left.urdf (robot description, URDF)
Before this commit: robot robotera_xhand_left, 23 links, 22 joints
Joints:
- joint left_hand_mid_joint3: origin xyz=0 0 -0.0424999999999995 rpy=0 0 0 -> xyz=0 -0.0008 -0.0424999999999995 rpy=0 0 0
- joint left_hand_thumb_rota_joint3: origin xyz=0.0504017317642718 0 0 rpy=0 0 0 -> xyz=0.0504017317642718 0 -0.0010 rpy=-1.570796 0 1.570796

File: src/robotera_ball_handling/source/robotera_ball_handling/assets/robots/xhand/urdf/robotera_xhand_right.urdf (robot description, URDF)
Before this commit: robot robotera_xhand_right, 23 links, 22 joints
Joints:
- joint right_hand_mid_joint3: origin xyz=0 0 -0.042107 rpy=0 0 0 -> xyz=0 0.0008 -0.042107 rpy=0 0 0
- joint right_hand_thumb_rota_joint3: origin xyz=0.0504024546888781 0 0 rpy=0 0 0 -> xyz=0.0504024546888781 0 -0.0010 rpy=-1.570796 0 1.570796
